File: KiCad/XIAO-ESP32-S3-PCB/XIAO-ESP32-S3-PCB.kicad_pcb (KiCad board)
At the start: 2 copper layers, 12 parts, among them J1 SK-3296S-01-L1, J2 A2001WR-S-2P_SMT, U1 XIAO-ESP32-S3-SMD

Commit message: hardware tested
Parts:
- removed J1: SK-3296S-01-L1, KiCad-switch:SK3296S01L1
- added SW1: SK-3296S-01-L1, Switch:SW-SMD_3P-P1.50_L2.7-W6.6, F.Cu at (130.0, 67.5)
Connections:
- U1 pad 10: PUSH_2 -> PUSH_1
- U1 pad 9: PUSH_1 -> PUSH_2
Routing:
- net PUSH_1: track 17.2 -> 21.5 mm
- net PUSH_2: track 26.0 -> 29.7 mm
- net 3V3: track 46.3 -> 43.7 mm
- net V_BATT: track 25.2 -> 27.1 mm
- net SWITCH_V_BATT: track 23.9 -> 24.5 mm
- added copper zone on F.Cu, net GND
