File: KiCad/XIAO-ESP32-S3-PCB/XIAO-ESP32-S3-PCB.kicad_sch (KiCad schematic)
At the start: 8 parts, among them J1 SK-3296S-01-L1, J2 A2001WR-S-2P_SMT, U1 XIAO-ESP32-S3-SMD

Commit message: hardware tested
Parts:
- removed J1: SK-3296S-01-L1, SK3296S01L1, symbol SK-3296S-01-L1:SK-3296S-01-L1
- added SW1: SK-3296S-01-L1, Switch:SW-SMD_3P-P1.50_L2.7-W6.6, symbol SCH_Switch-XIAO:SK-3296S-01-L1
Connections:
- net GND: now also SW1.0
- net PUSH_1: now also U1.10 (GPIO8_A9_D9_MISO); no longer U1.9 (GPIO7_A8_D8_SCK)
- net PUSH_2: now also U1.9 (GPIO7_A8_D8_SCK); no longer U1.10 (GPIO8_A9_D9_MISO)
- net SWITCH_V_BATT: now also SW1.1
- net V_BATT: now also SW1.2, SW1.3
